Commit message: Add phone_to_rebearm
1. phone_to_rebearm
2. Change urdf and xtl of OMX

File: examples/phone_to_omx/urdf/robot.urdf (robot description, URDF)
Before this commit: robot so101_new_calib, 8 links, 7 joints
Links:
- removed link base_link
- removed link gripper_frame_link
- removed link gripper_link
- removed link lower_arm_link
- removed link moving_jaw_so101_v1_link
- removed link shoulder_link
- removed link upper_arm_link
- removed link wrist_link
- added link end_effector_link; visual box size=0.01 0.01 0.01
- added link link0, mass 2.238905100e-01; collision mesh filename=assets/follower_01_base.stl scale=0.001 0.001 0.001; visual mesh filename=assets/follower_01_base.stl scale=0.001 0.001 0.001
- added link link1, mass 6.598704100e-02; collision mesh filename=assets/follower_02_base_tilt_Revised.stl scale=0.001 0.001 0.001; visual mesh filename=assets/follower_02_base_tilt_Revised.stl scale=0.001 0.001 0.001
- added link link2, mass 8.722147100e-02; collision mesh filename=assets/follower_03_middle_verticle.stl scale=0.001 0.001 0.001; visual mesh filename=assets/follower_03_middle_verticle.stl scale=0.001 0.001 0.001
- added link link3, mass 8.375912900e-02; collision mesh filename=assets/follower_04_middle_horizontal.stl scale=0.001 0.001 0.001; visual mesh filename=assets/follower_04_middle_horizontal.stl scale=0.001 0.001 0.001
- added link link4, mass 2.997506300e-02; collision mesh filename=assets/follower_05_tip.stl scale=0.001 0.001 0.001; visual mesh filename=assets/follower_05_tip.stl scale=0.001 0.001 0.001
- added link link5, mass 4.381088700e-02; collision mesh filename=assets/follower_06_pan_Revised.stl scale=0.001 0.001 0.001; visual mesh filename=assets/follower_06_pan_Revised.stl scale=0.001 0.001 0.001
- added link link6, mass 1.209067700e-02; collision mesh filename=assets/follower_07_gripper_motorized.stl scale=0.001 0.001 0.001; visual mesh filename=assets/follower_07_gripper_motorized.stl scale=0.001 0.001 0.001
- added link link7, mass 1.209067700e-02; collision mesh filename=assets/follower_08_gripper_gear.stl scale=0.001 0.001 0.001; visual mesh filename=assets/follower_08_gripper_gear.stl scale=0.001 0.001 0.001
- added link world
Joints:
- removed joint elbow_flex
- removed joint gripper
- removed joint gripper_frame_joint
- removed joint shoulder_lift
- removed joint shoulder_pan
- removed joint wrist_flex
- removed joint wrist_roll
- added joint end_effector_joint: type fixed, parent link5, child end_effector_link, origin xyz=0.09193 -0.0016 0 rpy=0 0 0
- added joint gripper_joint_1: type revolute, parent link5, child link6, origin xyz=0.0295 0.0075 0 rpy=0 0 0, axis 0 0 1, limit lower=-6.283185307179586 upper=6.283185307179586 effort=1000 velocity=4.8
- added joint gripper_joint_2: type revolute, parent link5, child link7, origin xyz=0.0295 -0.0108 0 rpy=0 0 0, axis 0 0 1, limit lower=-6.283185307179586 upper=6.283185307179586 effort=1000 velocity=4.8, mimic joint=gripper_joint_1 multiplier=-1
- added joint joint1: type revolute, parent link0, child link1, origin xyz=-0.01125 0 0.034 rpy=0 0 0, axis 0 0 1, limit lower=-6.283185307179586 upper=6.283185307179586 effort=1000 velocity=4.8
- added joint joint2: type revolute, parent link1, child link2, origin xyz=0 0 0.0635 rpy=0 0 0, axis 0 1 0, limit lower=-6.283185307179586 upper=6.283185307179586 effort=1000 velocity=4.8
- added joint joint3: type revolute, parent link2, child link3, origin xyz=0.0415 0 0.11315 rpy=0 0 0, axis 0 1 0, limit lower=-6.283185307179586 upper=6.283185307179586 effort=1000 velocity=4.8
- added joint joint4: type revolute, parent link3, child link4, origin xyz=0.162 0 0 rpy=0 0 0, axis 0 1 0, limit lower=-6.283185307179586 upper=6.283185307179586 effort=1000 velocity=4.8
- added joint joint5: type revolute, parent link4, child link5, origin xyz=0.0287 0 0 rpy=0 0 0, axis 1 0 0, limit lower=-6.283185307179586 upper=6.283185307179586 effort=1000 velocity=4.8
- added joint world_fixed: type fixed, parent world, child link0, origin xyz=0.0 0.0 0.0 rpy=0 0 0
